File: board/board_revA.brd (EAGLE design)
At the start: 94 x 44.5 mm, 69 parts, among them Q2 ULN2003AD, Y1 8Mhz

Commit message: [Board Rev A] Tweaking resistor values
Parts:
- R13: value 1K -> 2.2K
- R30, R32, R4, R6, R7: value 10K -> 470K 0.1%
- R31: value 1K -> 470K 0.1%
- R5: value 10K -> 100K
- R8: value 47K -> 470K 0.1%
Changed lines of the file:
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@@
 <attribute name="VALUE" x="61.79" y="11.5705" size="1.27" layer="28" rot="MR0"/>
 </element>
-<element name="R30" library="SparkFun-Resistors" package="0603-RES" value="10K" x="71.695" y="31.5525" smashed="yes" rot="MR90">
+<element name="R30" library="SparkFun-Resistors" package="0603-RES" value="470K 0.1%" x="71.695" y="31.5525" smashed="yes" rot="MR90">
 <attribute name="NAME" x="68.8935" y="35.0605" size="1.778" layer="26" font="vector" ratio="16" rot="MR180"/>
 <attribute name="VALUE" x="70.552" y="30.5365" size="0.4064" layer="28" font="vector" rot="MR90"/>
 </element>
-<element name="R31" library="SparkFun-Resistors" package="0603-RES" value="1K" x="75.98" y="24.8975" smashed="yes" rot="MR0">
+<element name="R31" library="SparkFun-Resistors" package="0603-RES" value="470K 0.1%" x="75.98" y="24.8975" smashed="yes" rot="MR0">
 <attribute name="NAME" x="77.404" y="22.222" size="1.778" layer="26" font="vector" ratio="16" rot="MR0"/>
 <attribute name="VALUE" x="76.996" y="23.7545" size="0.4064" layer="28" font="vector" rot="MR0"/>
 </element>
-<element name="R32" library="SparkFun-Resistors" package="0603-RES" value="10K" x="58.6475" y="6.5125" smashed="yes" rot="MR90">
+<element name="R32" library="SparkFun-Resistors" package="0603-RES" value="470K 0.1%" x="58.6475" y="6.5125" smashed="yes" rot="MR90">
 <attribute name="NAME" x="59.392" y="4.7785" size="1.778" layer="26" font="vector" ratio="16" rot="MR90"/>
 <attribute name="VALUE" x="57.5045" y="5.4965" size="0.4064" layer="28" font="vector" rot="MR90"/>
@@
 <attribute name="VALUE" x="8.726" y="19.6345" size="0.4064" layer="28" font="vector" rot="MR0"/>
 </element>
-<element name="R4" library="SparkFun-Resistors" package="0603-RES" value="10K" x="67.155" y="5.5325" smashed="yes" rot="MR90">
+<element name="R4" library="SparkFun-Resistors" package="0603-RES" value="470K 0.1%" x="67.155" y="5.5325" smashed="yes" rot="MR90">
 <attribute name="NAME" x="67.917" y="4.6435" size="1.778" layer="26" font="vector" ratio="16" rot="MR90"/>
 <attribute name="VALUE" x="66.012" y="4.5165" size="0.4064" layer="28" font="vector" rot="MR90"/>
 </element>
-<element name="R6" library="SparkFun-Resistors" package="0603-RES" value="10K" x="54.63" y="6.53" smashed="yes" rot="MR90">
+<element name="R6" library="SparkFun-Resistors" package="0603-RES" value="470K 0.1%" x="54.63" y="6.53" smashed="yes" rot="MR90">
 <attribute name="NAME" x="55.859" y="8.392" size="1.778" layer="26" font="vector" ratio="16" rot="MR0"/>
 <attribute name="VALUE" x="53.487" y="5.514" size="0.4064" layer="28" font="vector" rot="MR90"/>
 </element>
-<element name="R7" library="SparkFun-Resistors" package="0603-RES" value="10K" x="63.6975" y="6.08" smashed="yes" rot="MR180">
+<element name="R7" library="SparkFun-Resistors" package="0603-RES" value="470K 0.1%" x="63.6975" y="6.08" smashed="yes" rot="MR180">
 <attribute name="NAME" x="62.8085" y="5.318" size="1.778" layer="26" font="vector" ratio="16" rot="MR180"/>
 <attribute name="VALUE" x="62.6815" y="7.223" size="0.4064" layer="28" font="vector" rot="MR180"/>
@@
 <attribute name="VALUE" x="62.71" y="-1.2425" size="1.27" layer="27"/>
 </element>
-<element name="R5" library="SparkFun-Resistors" package="0603-RES" value="10K" x="47.3275" y="2.2525" smashed="yes" rot="MR270">
+<element name="R5" library="SparkFun-Resistors" package="0603-RES" value="100K" x="47.3275" y="2.2525" smashed="yes" rot="MR270">
 <attribute name="NAME" x="48.3155" y="7.3915" size="1.778" layer="26" font="vector" ratio="16" rot="MR270"/>
 <attribute name="VALUE" x="48.4705" y="3.2685" size="0.4064" layer="28" font="vector" rot="MR270"/>
@@
 <attribute name="VALUE" x="41.297" y="1.179" size="0.4064" layer="28" font="vector" rot="MR90"/>
 </element>
-<element name="R8" library="SparkFun-Resistors" package="0603-RES" value="47K" x="45.02" y="2.195" smashed="yes" rot="MR90">
+<element name="R8" library="SparkFun-Resistors" package="0603-RES" value="470K 0.1%" x="45.02" y="2.195" smashed="yes" rot="MR90">
 <attribute name="NAME" x="44.282" y="4.056" size="1.778" layer="26" font="vector" ratio="16" rot="MR90"/>
 <attribute name="VALUE" x="43.877" y="1.179" size="0.4064" layer="28" font="vector" rot="MR90"/>
@@
 <attribute name="NAME" x="20.27" y="29" size="1.778" layer="26" font="vector" ratio="16" rot="MR0"/>
 </element>
-<element name="R13" library="SparkFun-Resistors" package="0603-RES" value="1K" x="9.5" y="24.25" smashed="yes" rot="MR0">
+<element name="R13" library="SparkFun-Resistors" package="0603-RES" value="2.2K" x="9.5" y="24.25" smashed="yes" rot="MR0">
 <attribute name="NAME" x="11.389" y="25.012" size="1.778" layer="26" font="vector" ratio="16" rot="MR0"/>
 <attribute name="VALUE" x="10.516" y="23.107" size="0.4064" layer="28" font="vector" rot="MR0"/>

Commit message: [Board Rev A] Tweaking capacitor values
Parts:
- C1: value 4.7uF -> 1uF 25V
- C5, C7: value 4.7pF -> 33pF
- R30, R31, R32, R4, R6, R7: value 470K 0.1% -> 1M 1%
- R8: value 470K 0.1% -> 470K
- Y1: value 8Mhz -> 8Mhz 20pF
Changed lines of the file:
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@@
 <attribute name="VALUE" x="93.6225" y="30.585" size="1.27" layer="28" rot="MR270"/>
 </element>
-<element name="C1" library="SparkFun-Passives" package="0603-CAP" value="4.7uF" x="93.1425" y="33.16" smashed="yes" rot="MR270">
+<element name="C1" library="SparkFun-Passives" package="0603-CAP" value="1uF 25V" x="93.1425" y="33.16" smashed="yes" rot="MR270">
 <attribute name="NAME" x="93.8955" y="31.5515" size="1.778" layer="26" font="vector" ratio="16" rot="MR270"/>
 <attribute name="VALUE" x="94.2855" y="34.176" size="0.4064" layer="28" font="vector" rot="MR270"/>
@@
 <attribute name="VALUE" x="61.79" y="11.5705" size="1.27" layer="28" rot="MR0"/>
 </element>
-<element name="R30" library="SparkFun-Resistors" package="0603-RES" value="470K 0.1%" x="71.695" y="31.5525" smashed="yes" rot="MR90">
+<element name="R30" library="SparkFun-Resistors" package="0603-RES" value="1M 1%" x="71.695" y="31.5525" smashed="yes" rot="MR90">
 <attribute name="NAME" x="68.8935" y="35.0605" size="1.778" layer="26" font="vector" ratio="16" rot="MR180"/>
 <attribute name="VALUE" x="70.552" y="30.5365" size="0.4064" layer="28" font="vector" rot="MR90"/>
 </element>
-<element name="R31" library="SparkFun-Resistors" package="0603-RES" value="470K 0.1%" x="75.98" y="24.8975" smashed="yes" rot="MR0">
+<element name="R31" library="SparkFun-Resistors" package="0603-RES" value="1M 1%" x="75.98" y="24.8975" smashed="yes" rot="MR0">
 <attribute name="NAME" x="77.404" y="22.222" size="1.778" layer="26" font="vector" ratio="16" rot="MR0"/>
 <attribute name="VALUE" x="76.996" y="23.7545" size="0.4064" layer="28" font="vector" rot="MR0"/>
 </element>
-<element name="R32" library="SparkFun-Resistors" package="0603-RES" value="470K 0.1%" x="58.6475" y="6.5125" smashed="yes" rot="MR90">
+<element name="R32" library="SparkFun-Resistors" package="0603-RES" value="1M 1%" x="58.6475" y="6.5125" smashed="yes" rot="MR90">
 <attribute name="NAME" x="59.392" y="4.7785" size="1.778" layer="26" font="vector" ratio="16" rot="MR90"/>
 <attribute name="VALUE" x="57.5045" y="5.4965" size="0.4064" layer="28" font="vector" rot="MR90"/>
@@
 <attribute name="VALUE" x="8.726" y="19.6345" size="0.4064" layer="28" font="vector" rot="MR0"/>
 </element>
-<element name="R4" library="SparkFun-Resistors" package="0603-RES" value="470K 0.1%" x="67.155" y="5.5325" smashed="yes" rot="MR90">
+<element name="R4" library="SparkFun-Resistors" package="0603-RES" value="1M 1%" x="67.155" y="5.5325" smashed="yes" rot="MR90">
 <attribute name="NAME" x="67.917" y="4.6435" size="1.778" layer="26" font="vector" ratio="16" rot="MR90"/>
 <attribute name="VALUE" x="66.012" y="4.5165" size="0.4064" layer="28" font="vector" rot="MR90"/>
 </element>
-<element name="R6" library="SparkFun-Resistors" package="0603-RES" value="470K 0.1%" x="54.63" y="6.53" smashed="yes" rot="MR90">
+<element name="R6" library="SparkFun-Resistors" package="0603-RES" value="1M 1%" x="54.63" y="6.53" smashed="yes" rot="MR90">
 <attribute name="NAME" x="55.859" y="8.392" size="1.778" layer="26" font="vector" ratio="16" rot="MR0"/>
 <attribute name="VALUE" x="53.487" y="5.514" size="0.4064" layer="28" font="vector" rot="MR90"/>
 </element>
-<element name="R7" library="SparkFun-Resistors" package="0603-RES" value="470K 0.1%" x="63.6975" y="6.08" smashed="yes" rot="MR180">
+<element name="R7" library="SparkFun-Resistors" package="0603-RES" value="1M 1%" x="63.6975" y="6.08" smashed="yes" rot="MR180">
 <attribute name="NAME" x="62.8085" y="5.318" size="1.778" layer="26" font="vector" ratio="16" rot="MR180"/>
 <attribute name="VALUE" x="62.6815" y="7.223" size="0.4064" layer="28" font="vector" rot="MR180"/>
@@
 <attribute name="VALUE" x="41.297" y="1.179" size="0.4064" layer="28" font="vector" rot="MR90"/>
 </element>
-<element name="R8" library="SparkFun-Resistors" package="0603-RES" value="470K 0.1%" x="45.02" y="2.195" smashed="yes" rot="MR90">
+<element name="R8" library="SparkFun-Resistors" package="0603-RES" value="470K" x="45.02" y="2.195" smashed="yes" rot="MR90">
 <attribute name="NAME" x="44.282" y="4.056" size="1.778" layer="26" font="vector" ratio="16" rot="MR90"/>
 <attribute name="VALUE" x="43.877" y="1.179" size="0.4064" layer="28" font="vector" rot="MR90"/>
@@
 <attribute name="VALUE" x="3.901" y="20.754" size="0.4064" layer="28" rot="MR90"/>
 </element>
-<element name="Y1" library="SparkFun-FreqCtrl" package="HC49US" value="8Mhz" x="32" y="34.25" smashed="yes" rot="MR0">
+<element name="Y1" library="SparkFun-FreqCtrl" package="HC49US" value="8Mhz 20pF" x="32" y="34.25" smashed="yes" rot="MR0">
 <attribute name="NAME" x="33.465" y="29.794" size="1.778" layer="26" font="vector" ratio="16" rot="MR0"/>
 <attribute name="VALUE" x="37.715" y="30.059" size="1.27" layer="28" ratio="10" rot="MR0"/>
 </element>
-<element name="C5" library="SparkFun-Capacitors" package="0603-CAP" value="4.7pF" x="39" y="34.25" smashed="yes" rot="MR270">
+<element name="C5" library="SparkFun-Capacitors" package="0603-CAP" value="33pF" x="39" y="34.25" smashed="yes" rot="MR270">
 <attribute name="NAME" x="40.389" y="30.762" size="1.778" layer="26" font="vector" ratio="16" rot="MR0"/>
 <attribute name="VALUE" x="40.143" y="35.266" size="0.4064" layer="28" font="vector" rot="MR270"/>
 </element>
-<element name="C7" library="SparkFun-Capacitors" package="0603-CAP" value="4.7pF" x="25" y="34.25" smashed="yes" rot="MR270">
+<element name="C7" library="SparkFun-Capacitors" package="0603-CAP" value="33pF" x="25" y="34.25" smashed="yes" rot="MR270">
 <attribute name="NAME" x="23.111" y="32.488" size="1.778" layer="26" font="vector" ratio="16" rot="MR180"/>
 <attribute name="VALUE" x="26.143" y="35.266" size="0.4064" layer="28" font="vector" rot="MR270"/>
