File: board/board_revA.brd (EAGLE design)
At the start: 94 x 44.5 mm, 69 parts, among them Q2 ULN2003AD, Y1 8Mhz 20pF

Commit message: [GUI/Code] Rewrote DSP functions, switched to float; Updated DSP library
Parts:
- IC_OPA: value MCP6004 -> TL974IPW
Changed lines of the file:
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@@
 <?xml version="1.0" encoding="utf-8"?>
 <!DOCTYPE eagle SYSTEM "eagle.dtd">
-<eagle version="6.5.0">
+<eagle version="7.1.0">
 <drawing>
 <settings>
@@
 <pass name="Default">
 <param name="RoutingGrid" value="50mil"/>
+<param name="AutoGrid" value="1"/>
+<param name="Efforts" value="0"/>
+<param name="TopRouterVariant" value="1"/>
 <param name="tpViaShape" value="round"/>
 <param name="PrefDir.1" value="|"/>
@@
 <attribute name="VALUE" x="23.0725" y="11.09" size="1.27" layer="28" rot="MR180"/>
 </element>
-<element name="IC_OPA" library="linear" package="TSSOP14" value="MCP6004" x="59.885" y="15.5075" smashed="yes" rot="MR270">
+<element name="IC_OPA" library="linear" package="TSSOP14" value="TL974IPW" x="59.885" y="15.5075" smashed="yes" rot="MR270">
 <attribute name="NAME" x="54.3375" y="12.6755" size="1.778" layer="26" font="vector" ratio="16" rot="MR180"/>
 <attribute name="VALUE" x="61.79" y="11.5705" size="1.27" layer="28" rot="MR0"/>

Commit message: [Board A] Fixed resistor values
Parts:
- R31: value 1M 1% -> 100K 1%
Changed lines of the file:
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@@
 <attribute name="VALUE" x="70.552" y="30.5365" size="0.4064" layer="28" font="vector" rot="MR90"/>
 </element>
-<element name="R31" library="SparkFun-Resistors" package="0603-RES" value="1M 1%" x="75.98" y="24.8975" smashed="yes" rot="MR0">
+<element name="R31" library="SparkFun-Resistors" package="0603-RES" value="100K 1%" x="75.98" y="24.8975" smashed="yes" rot="MR0">
 <attribute name="NAME" x="77.404" y="22.222" size="1.778" layer="26" font="vector" ratio="16" rot="MR0"/>
 <attribute name="VALUE" x="76.996" y="23.7545" size="0.4064" layer="28" font="vector" rot="MR0"/>
