File: board/board_revB.sch (EAGLE design)
At the start: 65 parts, among them Q2 ULN2003AD, Y1 8Mhz

Commit message: [Board Rev B] Changed switch to a more common model using metric pitch
Parts:
- S1: value (none) -> EG1213; device SparkFun-Electromechanical:SWITCH-SPDTPTH -> adafruit:EG1213
Connections:
- net BUT1: now also S11.P; no longer S1.P
- net GND: now also S11.S; no longer S1.S
Changed lines of the file:
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@@
 <part name="R32" library="SparkFun-Resistors" deviceset="RESISTOR" device="0603-RES" value="10K"/>
 <part name="C34" library="SparkFun-Passives" deviceset="CAP" device="0603-CAP" value="4.7uF"/>
-<part name="S1" library="SparkFun-Electromechanical" deviceset="SWITCH-SPDT" device="PTH"/>
+<part name="S1" library="adafruit" deviceset="EG1213" device=""/>
 <part name="IC_CAN" library="SparkFun-DigitalIC" deviceset="MCP2551" device="" value="MAX3051"/>
 <part name="R3" library="SparkFun-Resistors" deviceset="RESISTOR" device="0603-RES" value="100K"/>
@@
 <instance part="R32" gate="G$1" x="36.83" y="120.65"/>
 <instance part="C34" gate="G$1" x="74.93" y="17.78"/>
-<instance part="S1" gate="1" x="77.47" y="59.69"/>
+<instance part="S1" gate="1" x="77.47" y="59.69" rot="R270"/>
 <instance part="IC_CAN" gate="G$1" x="300.99" y="82.55"/>
 <instance part="R3" gate="G$1" x="321.31" y="101.6" rot="R90"/>
@@
 <net name="BUT1" class="0">
 <segment>
-<wire x1="74.93" y1="59.69" x2="68.58" y2="59.69" width="0.1524" layer="91"/>
+<wire x1="72.39" y1="59.69" x2="68.58" y2="59.69" width="0.1524" layer="91"/>
 <label x="63.5" y="59.69" size="1.778" layer="95"/>
 <pinref part="C22" gate="G$1" pin="1"/>

Commit message: [GUI] Adding translation support
Parts:
- added CON_UART: (no value), SparkFun-Connectors:M03PTH
- added Q1: ULN2003AS, misc:ULN2003AS
Connections:
- new net UART_RXD_OUT: CON_UART.2, Q1.I1
- new net UART_TXD_OUT: CON_UART.3, Q1.O7
- net GND: now also CON_UART.1, Q1.GND
- net UART_RXD: now also Q1.O1
- net UART_TXD: now also Q1.I7
Changed lines of the file:
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@@
 <part name="R14" library="SparkFun-Resistors" deviceset="RESISTOR" device="0603-RES" value="0R"/>
 <part name="F1" library="misc" deviceset="PTC" device="1812K" value="24V 0.75A"/>
+<part name="Q1" library="misc" deviceset="ULN2003A" device="S" value="ULN2003AS"/>
+<part name="GND21" library="supply1" deviceset="GND" device=""/>
+<part name="CON_UART" library="SparkFun-Connectors" deviceset="M03" device="PTH"/>
+<part name="GND22" library="supply1" deviceset="GND" device=""/>
 </parts>
 <sheets>
@@
 <instance part="R14" gate="G$1" x="80.01" y="36.83" rot="R180"/>
 <instance part="F1" gate="G$1" x="39.37" y="36.83" rot="R90"/>
+<instance part="Q1" gate="A" x="304.8" y="180.34"/>
+<instance part="GND21" gate="1" x="292.1" y="167.64"/>
+<instance part="CON_UART" gate="G$1" x="285.75" y="156.21"/>
+<instance part="GND22" gate="1" x="293.37" y="151.13"/>
 </instances>
 <busses>
@@
 <pinref part="GND18" gate="1" pin="GND"/>
 </segment>
+<segment>
+<pinref part="Q1" gate="A" pin="GND"/>
+<pinref part="GND21" gate="1" pin="GND"/>
+</segment>
+<segment>
+<pinref part="CON_UART" gate="G$1" pin="1"/>
+<pinref part="GND22" gate="1" pin="GND"/>
+</segment>
 </net>
 <net name="+3V3" class="0">
@@
 <pinref part="STM32" gate="PORTA_H" pin="PA10"/>
 </segment>
+<segment>
+<pinref part="Q1" gate="A" pin="O1"/>
+<wire x1="317.5" y1="187.96" x2="332.74" y2="187.96" width="0.1524" layer="91"/>
+<label x="318.77" y="187.96" size="1.778" layer="95"/>
+</segment>
 </net>
 <net name="UART_TXD" class="0">
@@
 <label x="142.24" y="110.49" size="1.778" layer="95" rot="R180"/>
 <pinref part="STM32" gate="PORTA_H" pin="PA9"/>
+</segment>
+<segment>
+<pinref part="Q1" gate="A" pin="I7"/>
+<wire x1="292.1" y1="172.72" x2="278.13" y2="172.72" width="0.1524" layer="91"/>
+<label x="292.1" y="172.72" size="1.778" layer="95" rot="R180"/>
 </segment>
 </net>
@@
 </segment>
 </net>
+<net name="UART_RXD_OUT" class="0">
+<segment>
+<pinref part="Q1" gate="A" pin="I1"/>
+<wire x1="292.1" y1="187.96" x2="278.13" y2="187.96" width="0.1524" layer="91"/>
+<label x="292.1" y="187.96" size="1.778" layer="95" rot="R180"/>
+</segment>
+<segment>
+<pinref part="CON_UART" gate="G$1" pin="2"/>
+<wire x1="293.37" y1="156.21" x2="306.07" y2="156.21" width="0.1524" layer="91"/>
+<label x="293.37" y="156.21" size="1.778" layer="95"/>
+</segment>
+</net>
+<net name="UART_TXD_OUT" class="0">
+<segment>
+<pinref part="Q1" gate="A" pin="O7"/>
+<wire x1="317.5" y1="172.72" x2="331.47" y2="172.72" width="0.1524" layer="91"/>
+<label x="318.77" y="172.72" size="1.778" layer="95"/>
+</segment>
+<segment>
+<pinref part="CON_UART" gate="G$1" pin="3"/>
+<wire x1="293.37" y1="158.75" x2="306.07" y2="158.75" width="0.1524" layer="91"/>
+<label x="293.37" y="158.75" size="1.778" layer="95"/>
+</segment>
+</net>

Commit message: [Board Rev B] Updated additional UART interface
Connections:
- new net USART3_RX: Q1.O1, STM32PORTC_H.PC11
- new net USART3_TX: Q1.I7, STM32PORTC_H.PC10
- net UART_RXD: no longer Q1.O1
- net UART_TXD: no longer Q1.I7
Changed lines of the file:
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@@
 <grid distance="0.05" unitdist="inch" unit="inch" style="lines" multiple="1" display="yes" altdistance="0.005" altunitdist="inch" altunit="inch"/>
 <layers>
-<layer number="1" name="Top" color="4" fill="1" visible="yes" active="no"/>
-<layer number="2" name="Route2" color="1" fill="3" visible="yes" active="no"/>
-<layer number="3" name="Route3" color="4" fill="3" visible="yes" active="no"/>
-<layer number="4" name="Route4" color="1" fill="4" visible="yes" active="no"/>
-<layer number="5" name="Route5" color="4" fill="4" visible="yes" active="no"/>
-<layer number="6" name="Route6" color="1" fill="8" visible="yes" active="no"/>
-<layer number="7" name="Route7" color="4" fill="8" visible="yes" active="no"/>
-<layer number="8" name="Route8" color="1" fill="2" visible="yes" active="no"/>
-<layer number="9" name="Route9" color="4" fill="2" visible="yes" active="no"/>
-<layer number="10" name="Route10" color="1" fill="7" visible="yes" active="no"/>
-<layer number="11" name="Route11" color="4" fill="7" visible="yes" active="no"/>
-<layer number="12" name="Route12" color="1" fill="5" visible="yes" active="no"/>
-<layer number="13" name="Route13" color="4" fill="5" visible="yes" active="no"/>
-<layer number="14" name="Route14" color="1" fill="6" visible="yes" active="no"/>
-<layer number="15" name="Route15" color="4" fill="6" visible="yes" active="no"/>
-<layer number="16" name="Bottom" color="1" fill="1" visible="yes" active="no"/>
-<layer number="17" name="Pads" color="2" fill="1" visible="yes" active="no"/>
-<layer number="18" name="Vias" color="2" fill="1" visible="yes" active="no"/>
-<layer number="19" name="Unrouted" color="6" fill="1" visible="yes" active="no"/>
-<layer number="20" name="Dimension" color="15" fill="1" visible="yes" active="no"/>
-<layer number="21" name="tPlace" color="16" fill="1" visible="yes" active="no"/>
-<layer number="22" name="bPlace" color="14" fill="1" visible="yes" active="no"/>
-<layer number="23" name="tOrigins" color="15" fill="1" visible="yes" active="no"/>
-<layer number="24" name="bOrigins" color="15" fill="1" visible="yes" active="no"/>
-<layer number="25" name="tNames" color="7" fill="1" visible="yes" active="no"/>
-<layer number="26" name="bNames" color="7" fill="1" visible="yes" active="no"/>
-<layer number="27" name="tValues" color="7" fill="1" visible="yes" active="no"/>
-<layer number="28" name="bValues" color="7" fill="1" visible="yes" active="no"/>
+<layer number="1" name="Top" color="4" fill="1" visible="no" active="no"/>
+<layer number="2" name="Route2" color="1" fill="3" visible="no" active="no"/>
+<layer number="3" name="Route3" color="4" fill="3" visible="no" active="no"/>
+<layer number="4" name="Route4" color="1" fill="4" visible="no" active="no"/>
+<layer number="5" name="Route5" color="4" fill="4" visible="no" active="no"/>
+<layer number="6" name="Route6" color="1" fill="8" visible="no" active="no"/>
+<layer number="7" name="Route7" color="4" fill="8" visible="no" active="no"/>
+<layer number="8" name="Route8" color="1" fill="2" visible="no" active="no"/>
+<layer number="9" name="Route9" color="4" fill="2" visible="no" active="no"/>
+<layer number="10" name="Route10" color="1" fill="7" visible="no" active="no"/>
+<layer number="11" name="Route11" color="4" fill="7" visible="no" active="no"/>
+<layer number="12" name="Route12" color="1" fill="5" visible="no" active="no"/>
+<layer number="13" name="Route13" color="4" fill="5" visible="no" active="no"/>
+<layer number="14" name="Route14" color="1" fill="6" visible="no" active="no"/>
+<layer number="15" name="Route15" color="4" fill="6" visible="no" active="no"/>
+<layer number="16" name="Bottom" color="1" fill="1" visible="no" active="no"/>
+<layer number="17" name="Pads" color="2" fill="1" visible="no" active="no"/>
+<layer number="18" name="Vias" color="2" fill="1" visible="no" active="no"/>
+<layer number="19" name="Unrouted" color="6" fill="1" visible="no" active="no"/>
+<layer number="20" name="Dimension" color="15" fill="1" visible="no" active="no"/>
+<layer number="21" name="tPlace" color="16" fill="1" visible="no" active="no"/>
+<layer number="22" name="bPlace" color="14" fill="1" visible="no" active="no"/>
+<layer number="23" name="tOrigins" color="15" fill="1" visible="no" active="no"/>
+<layer number="24" name="bOrigins" color="15" fill="1" visible="no" active="no"/>
+<layer number="25" name="tNames" color="7" fill="1" visible="no" active="no"/>
+<layer number="26" name="bNames" color="7" fill="1" visible="no" active="no"/>
+<layer number="27" name="tValues" color="7" fill="1" visible="no" active="no"/>
+<layer number="28" name="bValues" color="7" fill="1" visible="no" active="no"/>
 <layer number="29" name="tStop" color="7" fill="3" visible="no" active="no"/>
 <layer number="30" name="bStop" color="7" fill="6" visible="no" active="no"/>
@@
 <layer number="35" name="tGlue" color="7" fill="4" visible="no" active="no"/>
 <layer number="36" name="bGlue" color="7" fill="5" visible="no" active="no"/>
-<layer number="37" name="tTest" color="7" fill="1" visible="yes" active="no"/>
-<layer number="38" name="bTest" color="7" fill="1" visible="yes" active="no"/>
+<layer number="37" name="tTest" color="7" fill="1" visible="no" active="no"/>
+<layer number="38" name="bTest" color="7" fill="1" visible="no" active="no"/>
 <layer number="39" name="tKeepout" color="4" fill="11" visible="no" active="no"/>
 <layer number="40" name="bKeepout" color="1" fill="11" visible="no" active="no"/>
@@
 <layer number="44" name="Drills" color="7" fill="1" visible="no" active="no"/>
 <layer number="45" name="Holes" color="7" fill="1" visible="no" active="no"/>
-<layer number="46" name="Milling" color="3" fill="1" visible="yes" active="no"/>
-<layer number="47" name="Measures" color="7" fill="1" visible="yes" active="no"/>
-<layer number="48" name="Document" color="7" fill="1" visible="yes" active="no"/>
-<layer number="49" name="Reference" color="7" fill="1" visible="yes" active="no"/>
-<layer number="50" name="dxf" color="7" fill="1" visible="yes" active="no"/>
-<layer number="51" name="tDocu" color="6" fill="1" visible="yes" active="no"/>
-<layer number="52" name="bDocu" color="7" fill="1" visible="yes" active="no"/>
-<layer number="53" name="tGND_GNDA" color="7" fill="9" visible="yes" active="no"/>
-<layer number="54" name="bGND_GNDA" color="1" fill="9" visible="yes" active="no"/>
-<layer number="56" name="wert" color="7" fill="1" visible="yes" active="no"/>
-<layer number="57" name="tCAD" color="7" fill="1" visible="yes" active="no"/>
+<layer number="46" name="Milling" color="3" fill="1" visible="no" active="no"/>
+<layer number="47" name="Measures" color="7" fill="1" visible="no" active="no"/>
+<layer number="48" name="Document" color="7" fill="1" visible="no" active="no"/>
+<layer number="49" name="Reference" color="7" fill="1" visible="no" active="no"/>
+<layer number="50" name="dxf" color="7" fill="1" visible="no" active="no"/>
+<layer number="51" name="tDocu" color="6" fill="1" visible="no" active="no"/>
+<layer number="52" name="bDocu" color="7" fill="1" visible="no" active="no"/>
+<layer number="53" name="tGND_GNDA" color="7" fill="9" visible="no" active="no"/>
+<layer number="54" name="bGND_GNDA" color="1" fill="9" visible="no" active="no"/>
+<layer number="56" name="wert" color="7" fill="1" visible="no" active="no"/>
+<layer number="57" name="tCAD" color="7" fill="1" visible="no" active="no"/>
 <layer number="91" name="Nets" color="2" fill="1" visible="yes" active="yes"/>
 <layer number="92" name="Busses" color="1" fill="1" visible="yes" active="yes"/>
@@
 <pinref part="STM32" gate="PORTA_H" pin="PA10"/>
 </segment>
-<segment>
-<pinref part="Q1" gate="A" pin="O1"/>
-<wire x1="317.5" y1="187.96" x2="332.74" y2="187.96" width="0.1524" layer="91"/>
-<label x="318.77" y="187.96" size="1.778" layer="95"/>
-</segment>
 </net>
 <net name="UART_TXD" class="0">
@@
 <label x="142.24" y="110.49" size="1.778" layer="95" rot="R180"/>
 <pinref part="STM32" gate="PORTA_H" pin="PA9"/>
-</segment>
-<segment>
-<pinref part="Q1" gate="A" pin="I7"/>
-<wire x1="292.1" y1="172.72" x2="278.13" y2="172.72" width="0.1524" layer="91"/>
-<label x="292.1" y="172.72" size="1.778" layer="95" rot="R180"/>
 </segment>
 </net>
@@
 </segment>
 </net>
+<net name="USART3_TX" class="0">
+<segment>
+<pinref part="STM32" gate="PORTC_H" pin="PC10"/>
+<wire x1="142.24" y1="57.15" x2="127" y2="57.15" width="0.1524" layer="91"/>
+<label x="127" y="57.15" size="1.778" layer="95"/>
+</segment>
+<segment>
+<pinref part="Q1" gate="A" pin="I7"/>
+<wire x1="292.1" y1="172.72" x2="278.13" y2="172.72" width="0.1524" layer="91"/>
+<label x="292.1" y="172.72" size="1.778" layer="95" rot="R180"/>
+</segment>
+</net>
+<net name="USART3_RX" class="0">
+<segment>
+<pinref part="STM32" gate="PORTC_H" pin="PC11"/>
+<wire x1="142.24" y1="54.61" x2="127" y2="54.61" width="0.1524" layer="91"/>
+<label x="127" y="54.61" size="1.778" layer="95"/>
+</segment>
+<segment>
+<pinref part="Q1" gate="A" pin="O1"/>
+<wire x1="317.5" y1="187.96" x2="332.74" y2="187.96" width="0.1524" layer="91"/>
+<label x="318.77" y="187.96" size="1.778" layer="95"/>
+</segment>
+</net>
