File: board/board_revB.sch (EAGLE design)
At the start: 85 parts, among them IC1 MCP1703CB, Q2 ULN2003AD, U1 MAX202, Y1 8Mhz

Commit message: [Board] working on rev B (full rework)
Parts:
- removed C34: 4.7uF, SparkFun-Passives:CAP0603-CAP
- removed CON_AN, CON_KNK, CON_PWR, CON_RPM-VSS: (no value), SparkFun-Connectors:M03LOCK
- removed CON_CAN, CON_K-LINE, CON_UART1, CON_UART2: M02LOCK, SparkFun-Connectors:M02LOCK
- removed CON_USB: (no value), SparkFun-Connectors:M04LOCK
- removed D5: B240A, SparkFun-DiscreteSemi:DIODESMA
- removed IC1: MCP1703CB, linear:MCP1703CB
- removed IC_REG: LM1117-3.3, v-reg:LD117ADT33TR
- removed R10, R25, R26: 1K, SparkFun-Resistors:RESISTOR0603-RES
- removed R14: 0R, SparkFun-Resistors:RESISTOR0603-RES
- removed TVS2: NUP4201MR6, misc:NUP4201MR6
- added C14: 10nF, SparkFun-Capacitors:CAP0603-CAP
- added C9: 47uF 25v, SparkFun-Passives:CAP_POLPTH2
- added F2: 1206L020 24V 0.2A, misc:PTCSMD
- added JP1: USBSMD, SparkFun-Connectors:USBSMD
- added U2, U3: LDK120DM33R, SparkFun-PowerIC:V_REG_LDOSMD
- added VR1: LM2931, SparkFun-PowerIC:LM2931
- added X2: (no value), con-molex-micro-fit-3_0:HEADER_POS16_43045-1600
- C1: value 4.7uF -> 1uF
- CON_DBG: value (none) -> JST_VERTICAL; device SparkFun-Connectors:M03X22X3_SILK_SM -> SparkFun-Connectors:JST_VERTICAL
- D1: value B240A -> BAT165; device SparkFun-DiscreteSemi:DIODESMA -> SparkFun-DiscreteSemi:DIODESOD
- D6: value B240A -> BAT165
- F1: value 24V 0.75A -> 1206L020 24V 0.2A; device misc:PTC1812K -> misc:PTCSMD
- IC_OPA: value TL974IPW -> MCP6004
- R19, R20, R24: value 10K 1% -> 2K 1%
- R21, R22: value 56R -> 1K
- R23, R6, R7: value 10K 1% -> 1K 1%
- S1: value EG1213 -> SWITCH-MOMENTARY-2SMD-4; device adafruit:EG1213 -> SparkFun-Electromechanical:SWITCH-MOMENTARY-2SMD-4
- renumbered IC_FRAM to IC_EE
Connections:
- removed net N$1: CON_KNK.2, R1.1
- removed net N$12: CON_RPM-VSS.3, R25.1
- removed net N$14: C5.2, R14.1, Y1.1
- removed net N$16: Q2.I6, R25.2
- removed net N$18: C3.2, R10.1, R11.1
- removed net N$21: CON_RPM-VSS.2, R26.1
- removed net OP3_VINM: D4.C1A2, R5.2, R8.1, STM32PORTB_L.PB2
- removed net OP3_VOUT: R5.1, STM32PORTB_L.PB1
- removed net SWDAT: CON_DBG.6, STM32PORTA_H.PA13
- removed net UART2_RXD_OUT: CON_UART2.2, U1.R1IN
- removed net UART2_TXD_OUT: CON_UART2.1, U1.T1OUT
- removed net UART3_RXD_OUT: CON_UART1.2, U1.R2IN
- removed net UART3_TXD_OUT: CON_UART1.1, U1.T2OUT
- removed net USART2_RX: STM32PORTB_L.PB4, U1.R1OUT
- removed net USART2_TX: STM32PORTB_L.PB3, U1.T1IN
- removed net USART3_RX: STM32PORTC_H.PC11, U1.R2OUT
- removed net USART3_TX: STM32PORTC_H.PC10, U1.T2IN
- new net AN2_IN: R32.1, X2.8
- new net AN3_IN: R4.1, X2.7
- new net FREQ1_RAW: Q2.I6, X2.4
- new net FREQ2_RAW: Q2.I7, X2.12
- new net KNK_AN: IC_OPAD.OUT, R5.1, STM32PORTB_L.PB1
- new net KNK_BIAS: R1.1, X2.10
- new net KNK_IN: C4.1, X2.11
- new net N$32: C1.2, TVS1.1, VR1.GND@6, VR1.GND@7
- new net SWDIO: CON_DBG.4, STM32PORTA_H.PA13
- new net SWO: CON_DBG.6
- new net UART1_RXD_232: U1.R1IN, X2.2
- new net UART1_TXD_232: U1.T1OUT, X2.3
- new net UART2_RX: STM32PORTB_L.PB4, U1.R2OUT
- new net UART2_RXD_232: U1.R2IN
- new net UART2_TX: STM32PORTB_L.PB3, U1.T2IN
- new net UART2_TXD_232: U1.T2OUT
- new net UART3_RX: IC_KLINE.RXD@1, R2.1, STM32PORTC_H.PC11
- new net UART3_TX: IC_KLINE.TXD@4, STM32PORTC_H.PC10
- new net VDDA: C30.1, C31.1, STM32AN_POWER.VDDA, U3.OUT
- net +12V: now also X2.16; no longer CON_PWR.3
- net +3V3: now also S1.2, U2.OUT; no longer C13.1, C2.1, C30.1, C31.1, C34.1, IC_REG.OUT, LED1.A, LED2.A, R1.2, STM32AN_POWER.VDDA, TP2.P$1, U1.VCC
- net +5V: now also C13.1, C2.1, C9.+, LED1.A, LED2.A, R1.2, TP2.P$1, U1.VCC, U2.EN, U2.IN, U3.EN, U3.IN, VR1.OUT; no longer IC1.VO
- net AN2: now also STM32PORTC_L.PC2; no longer STM32PORTC_L.PC3
- net AN3: now also STM32PORTC_L.PC3; no longer STM32PORTC_L.PC2
- net BOOT0: now also S1.1
- net BUT1: now also S21.P; no longer S11.P
- net BUT2: no longer S21.P
- net CANH: now also X2.6; no longer CON_CAN.2
- net CANL: now also X2.5; no longer CON_CAN.1
- net DAC1: now also IC_OPAD.+IN
- net GND: now also C14.2, C9.-, CON_DBG.3, JP1.GND, U2.GND, U3.GND, VR1.GND@2, VR1.GND@3, X2.1, X2.15, X2.9; no longer C1.2, C34.2, CON_AN.1, CON_DBG.4, CON_KNK.1, CON_PWR.2, CON_RPM-VSS.1, CON_USB.4, IC1.GND, IC_OPAD.+IN, IC_OPAD.-IN, IC_REG.ADJ, S11.S, TVS1.1, TVS2.VN@2
- net K-LINE: now also X2.14; no longer CON_K-LINE.2
- net N$17: now also JP1.D-; no longer CON_USB.2, TVS2.IO@4
- net N$2: now also STM32PORTB_L.PB2; no longer CON_AN.3, R32.1
- net N$3: now also F2.1, Q2.O1; no longer CON_AN.2, R4.1
- net N$4: now also D4.C1A2, IC_OPAD.-IN, R5.2, R8.1; no longer C4.1, CON_KNK.3
- net N$7: now also JP1.D+; no longer CON_USB.1, TVS2.IO@3
- net N$9: now also C14.1, U3.BP; no longer Q2.I7, R26.2
- net NRST: now also C3.2, CON_DBG.5, R11.1; no longer CON_DBG.3, R10.2
- net OSC_OUT: now also C5.2, Y1.1; no longer R14.2
- net RELAY_OUT: now also F2.2; no longer CON_PWR.1, Q2.O1
- net SCS: now also X2.13; no longer CON_K-LINE.1
- net UART1_RX: now also U1.R1OUT; no longer IC_KLINE.RXD@1, R2.1
- net UART1_TX: now also U1.T1IN; no longer IC_KLINE.TXD@4
- net USB_VBUS: now also JP1.VBUS; no longer CON_USB.3, D5.A, TVS2.VBUS@5
- net VCC: no longer D5.C
- net VCC_PROT: now also VR1.IN; no longer IC1.VI, IC_REG.IN
Other:
- note added: "Same pinout as Discovery boards"
- moved on the sheet: C1, C10, C11, C2, C3, C4, C5, C7, D1, D4, F1, IC_OPAD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

Commit message: [Board] working on rev B (routing)
Parts:
- removed F2: 1206L020 24V 0.2A, misc:PTCSMD
- renumbered U1 to IC_232, U2 to VR2, U3 to VR3
Connections:
- removed net N$3: F2.1, Q2.O1
- removed net N$32: C1.2, TVS1.1, VR1.GND@6, VR1.GND@7
- removed net RELAY_OUT: F2.2
- net GND: now also C1.2, TVS1.1, VR1.GND@6, VR1.GND@7
- net RELAY_TRIG: no longer Q2.I1
- net UART1_RXD_232: now also X2.3; no longer X2.2
- net UART1_TXD_232: now also X2.2; no longer X2.3

Commit message: [Board] working on rev B (routing)
Parts:
- added D5: BAT165, SparkFun-DiscreteSemi:DIODESOD
- added JP2: (no value), SparkFun-Connectors:M03LOCK
Connections:
- net +5V: now also D5.C
- net GND: now also JP2.3
- net UART2_RXD_232: now also JP2.2
- net UART2_TXD_232: now also JP2.1
- net USB_VBUS: now also D5.A

Commit message: [Board] working on rev B (routing)
Connections:
- net DAC2 renamed SPI1_SCK
- net RELAY_TRIG renamed SPI1_MOSI
- removed net BUT2: STM32PORTC_H.PC13
- removed net N$2: STM32PORTB_L.PB2
- new net SPI1_MISO: STM32PORTA_L.PA6
- net BUT1: now also STM32POWER.VSS_4; no longer STM32PORTC_H.PC14
- net GND: no longer STM32POWER.VSS_4
- net LED1_TRIG: now also STM32PORTB_L.PB6; no longer STM32PORTA_L.PA2
- net LED2_TRIG: now also STM32PORTB_L.PB7; no longer STM32PORTA_L.PA3
Changed lines of the file:
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@@
 <layer number="230" name="230bmp" color="7" fill="1" visible="yes" active="yes"/>
 <layer number="231" name="231bmp" color="7" fill="1" visible="yes" active="yes"/>
+<layer number="232" name="Eagle3D_PG2" color="7" fill="1" visible="no" active="no"/>
+<layer number="233" name="Eagle3D_PG3" color="7" fill="1" visible="no" active="no"/>
 <layer number="248" name="Housing" color="7" fill="1" visible="yes" active="yes"/>
 <layer number="249" name="Edge" color="7" fill="1" visible="yes" active="yes"/>
@@
 <wire x1="176.53" y1="76.2" x2="176.53" y2="81.28" width="0.1524" layer="91"/>
 <junction x="176.53" y="76.2"/>
-<pinref part="STM32" gate="POWER" pin="VSS_4"/>
-<wire x1="176.53" y1="81.28" x2="176.53" y2="86.36" width="0.1524" layer="91"/>
-<junction x="176.53" y="81.28"/>
 <pinref part="GND10" gate="1" pin="GND"/>
 <junction x="176.53" y="71.12"/>
@@
 <net name="BUT1" class="0">
 <segment>
-<pinref part="STM32" gate="PORTC_H" pin="PC14"/>
-<wire x1="142.24" y1="46.99" x2="135.89" y2="46.99" width="0.1524" layer="91"/>
-<label x="142.24" y="46.99" size="1.778" layer="95" rot="R180"/>
-</segment>
-<segment>
 <wire x1="71.12" y1="48.26" x2="67.31" y2="48.26" width="0.1524" layer="91"/>
 <label x="62.23" y="48.26" size="1.778" layer="95"/>
 <wire x1="67.31" y1="48.26" x2="62.23" y2="48.26" width="0.1524" layer="91"/>
 <pinref part="S2" gate="1" pin="P"/>
+</segment>
+<segment>
+<pinref part="STM32" gate="POWER" pin="VSS_4"/>
+<wire x1="176.53" y1="86.36" x2="184.15" y2="86.36" width="0.1524" layer="91"/>
+<label x="176.53" y="86.36" size="1.778" layer="95"/>
 </segment>
 </net>
@@
 <net name="DAC1" class="0">
 <segment>
-<wire x1="142.24" y1="128.27" x2="134.62" y2="128.27" width="0.1524" layer="91"/>
+<wire x1="142.24" y1="128.27" x2="129.54" y2="128.27" width="0.1524" layer="91"/>
 <label x="142.24" y="128.27" size="1.778" layer="95" rot="R180"/>
 <pinref part="STM32" gate="PORTA_L" pin="PA4"/>
@@
 </segment>
 <segment>
-<pinref part="STM32" gate="PORTA_L" pin="PA2"/>
-<wire x1="142.24" y1="133.35" x2="134.62" y2="133.35" width="0.1524" layer="91"/>
-<label x="142.24" y="133.35" size="1.778" layer="95" rot="R180"/>
+<pinref part="STM32" gate="PORTB_L" pin="PB6"/>
+<wire x1="176.53" y1="123.19" x2="190.5" y2="123.19" width="0.1524" layer="91"/>
+<label x="176.53" y="123.19" size="1.778" layer="95"/>
 </segment>
 </net>
@@
 </segment>
 <segment>
-<pinref part="STM32" gate="PORTA_L" pin="PA3"/>
-<wire x1="142.24" y1="130.81" x2="134.62" y2="130.81" width="0.1524" layer="91"/>
-<label x="142.24" y="130.81" size="1.778" layer="95" rot="R180"/>
+<pinref part="STM32" gate="PORTB_L" pin="PB7"/>
+<wire x1="176.53" y1="120.65" x2="190.5" y2="120.65" width="0.1524" layer="91"/>
+<label x="176.53" y="120.65" size="1.778" layer="95"/>
 </segment>
 </net>
@@
 </segment>
 </net>
-<net name="RELAY_TRIG" class="0">
-<segment>
-<pinref part="STM32" gate="PORTA_L" pin="PA7"/>
-<wire x1="142.24" y1="120.65" x2="134.62" y2="120.65" width="0.1524" layer="91"/>
-<label x="142.24" y="120.65" size="1.778" layer="95" rot="R180"/>
-</segment>
-</net>
 <net name="USB_DETECT" class="0">
 <segment>
@@
 <wire x1="276.86" y1="66.04" x2="287.02" y2="66.04" width="0.1524" layer="91"/>
 <junction x="287.02" y="66.04"/>
-</segment>
-</net>
-<net name="BUT2" class="0">
-<segment>
-<wire x1="142.24" y1="49.53" x2="135.89" y2="49.53" width="0.1524" layer="91"/>
-<label x="142.24" y="49.53" size="1.778" layer="95" rot="R180"/>
-<pinref part="STM32" gate="PORTC_H" pin="PC13"/>
 </segment>
 </net>
@@
 </segment>
 </net>
-<net name="DAC2" class="0">
+<net name="SPI1_SCK" class="0">
 <segment>
 <pinref part="STM32" gate="PORTA_L" pin="PA5"/>
-<wire x1="142.24" y1="125.73" x2="134.62" y2="125.73" width="0.1524" layer="91"/>
+<wire x1="142.24" y1="125.73" x2="129.54" y2="125.73" width="0.1524" layer="91"/>
 <label x="142.24" y="125.73" size="1.778" layer="95" rot="R180"/>
 </segment>
@@
 </segment>
 </net>
-<net name="N$2" class="0">
-<segment>
-<pinref part="STM32" gate="PORTB_L" pin="PB2"/>
-<wire x1="176.53" y1="133.35" x2="190.5" y2="133.35" width="0.1524" layer="91"/>
-<label x="176.53" y="133.35" size="1.778" layer="95"/>
-</segment>
-</net>
 <net name="N$4" class="0">
 <segment>
@@
 </segment>
 </net>
+<net name="SPI1_MISO" class="0">
+<segment>
+<pinref part="STM32" gate="PORTA_L" pin="PA6"/>
+<wire x1="142.24" y1="123.19" x2="129.54" y2="123.19" width="0.1524" layer="91"/>
+<label x="142.24" y="123.19" size="1.778" layer="95" rot="R180"/>
+</segment>
+</net>
+<net name="SPI1_MOSI" class="0">
+<segment>
+<pinref part="STM32" gate="PORTA_L" pin="PA7"/>
+<wire x1="142.24" y1="120.65" x2="129.54" y2="120.65" width="0.1524" layer="91"/>
+<label x="142.24" y="120.65" size="1.778" layer="95" rot="R180"/>
+</segment>
+</net>

Commit message: [Board] working on rev B (routing)
Parts:
- removed CON_DBG: JST_VERTICAL, SparkFun-Connectors:JST_VERTICAL
- added JP4: (no value), SparkFun-Connectors:M05JST
Connections:
- removed net SWO: CON_DBG.6
- net +3V3: now also JP4.5; no longer CON_DBG.1
- net GND: now also JP4.3; no longer CON_DBG.3
- net NRST: now also JP4.1; no longer CON_DBG.5
- net SWCLK: now also JP4.4; no longer CON_DBG.2
- net SWDIO: now also JP4.2; no longer CON_DBG.4
Changed lines of the file:
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@@
 <part name="+3V1" library="supply1" deviceset="+3V3" device=""/>
 <part name="+3V3" library="supply1" deviceset="+3V3" device=""/>
-<part name="CON_DBG" library="SparkFun-Connectors" deviceset="JST_VERTICAL" device=""/>
 <part name="X2" library="con-molex-micro-fit-3_0" deviceset="HEADER_POS16_?" device="43045-1600"/>
 <part name="GND15" library="supply1" deviceset="GND" device=""/>
@@
 <part name="GND17" library="supply1" deviceset="GND" device=""/>
 <part name="D5" library="SparkFun-DiscreteSemi" deviceset="DIODE" device="SOD" value="BAT165"/>
+<part name="JP4" library="SparkFun-Connectors" deviceset="M05" device="JST"/>
 </parts>
 <sheets>
@@
 <instance part="+3V1" gate="G$1" x="53.34" y="55.88"/>
 <instance part="+3V3" gate="G$1" x="81.28" y="76.2"/>
-<instance part="CON_DBG" gate="G$1" x="250.19" y="133.35"/>
 <instance part="X2" gate="G$1" x="415.29" y="54.61" rot="MR180"/>
 <instance part="GND15" gate="1" x="62.23" y="205.74"/>
@@
 <attribute name="VALUE" x="127" y="219.4814" size="1.778" layer="96" rot="R180"/>
 </instance>
+<instance part="JP4" gate="G$1" x="245.11" y="133.35" rot="MR0"/>
 </instances>
 <busses>
@@
 </segment>
 <segment>
-<pinref part="CON_DBG" gate="G$1" pin="3"/>
 <wire x1="237.49" y1="133.35" x2="226.06" y2="133.35" width="0.1524" layer="91"/>
 <label x="237.49" y="133.35" size="1.778" layer="95" rot="R180"/>
+<pinref part="JP4" gate="G$1" pin="3"/>
 </segment>
 <segment>
@@
 </segment>
 <segment>
-<pinref part="CON_DBG" gate="G$1" pin="1"/>
 <wire x1="237.49" y1="138.43" x2="226.06" y2="138.43" width="0.1524" layer="91"/>
 <label x="237.49" y="138.43" size="1.778" layer="95" rot="R180"/>
+<pinref part="JP4" gate="G$1" pin="5"/>
 </segment>
 </net>
@@
 </segment>
 <segment>
-<pinref part="CON_DBG" gate="G$1" pin="5"/>
 <wire x1="237.49" y1="128.27" x2="226.06" y2="128.27" width="0.1524" layer="91"/>
 <label x="237.49" y="128.27" size="1.778" layer="95" rot="R180"/>
+<pinref part="JP4" gate="G$1" pin="1"/>
 </segment>
 </net>
@@
 </segment>
 <segment>
-<pinref part="CON_DBG" gate="G$1" pin="4"/>
 <wire x1="237.49" y1="130.81" x2="226.06" y2="130.81" width="0.1524" layer="91"/>
 <label x="237.49" y="130.81" size="1.778" layer="95" rot="R180"/>
+<pinref part="JP4" gate="G$1" pin="2"/>
 </segment>
 </net>
@@
 </segment>
 <segment>
-<pinref part="CON_DBG" gate="G$1" pin="2"/>
 <wire x1="237.49" y1="135.89" x2="226.06" y2="135.89" width="0.1524" layer="91"/>
 <label x="237.49" y="135.89" size="1.778" layer="95" rot="R180"/>
+<pinref part="JP4" gate="G$1" pin="4"/>
 </segment>
 </net>
@@
 </segment>
 </net>
-<net name="SWO" class="0">
-<segment>
-<pinref part="CON_DBG" gate="G$1" pin="6"/>
-<wire x1="237.49" y1="125.73" x2="226.06" y2="125.73" width="0.1524" layer="91"/>
-<label x="237.49" y="125.73" size="1.778" layer="95" rot="R180"/>
-</segment>
-</net>

Commit message: [Board] working on rev B (routing/schema)
Parts:
- C9: value 47uF 25v -> 100uF 16v
- IC_KLINE: value MCP2004 -> TJA1027
Connections:
- removed net N$7: JP1.D+, R15.1, R17.2
- net +12V: no longer D6.A, IC_KLINE.VBB@7
- net +3V3: now also R17.1
- net USB_CTRL: now also JP1.D+, R15.1, R17.2; no longer R17.1
- net VCC_PROT: now also D6.A, IC_KLINE.VBB@7

Commit message: [Board] working on rev B (routing/cleaning)
Parts:
- removed S2: EG1213, adafruit:EG1213
- added S3: SWITCH-MOMENTARY-2SIDE_EZ, SparkFun-Electromechanical:SWITCH-MOMENTARY-2SIDE_EZ
- JP1: value USBSMD -> USB-B; device SparkFun-Connectors:USBSMD -> SparkFun-Connectors:USBPTH
- renumbered JP2 to CON_RS232
Connections:
- new net VCC_DETECT: Q2.O1, STM32PORTB_L.PB5
- net BUT1: now also S3.1; no longer S21.P
- net GND: now also S3.2; no longer S21.S
- net VCC_PROT: now also Q2.I1
Changed lines of the file:
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@@
 <part name="GND21" library="supply1" deviceset="GND" device=""/>
 <part name="GND24" library="supply1" deviceset="GND" device=""/>
-<part name="S2" library="adafruit" deviceset="EG1213" device=""/>
 <part name="P+5" library="supply1" deviceset="+12V" device=""/>
 <part name="TP3" library="microbuilder" deviceset="TESTPOINT" device="ROUND1MM"/>
@@
 <part name="C9" library="SparkFun-Passives" deviceset="CAP_POL" device="PTH2" value="100uF 16v"/>
 <part name="S1" library="SparkFun-Electromechanical" deviceset="SWITCH-MOMENTARY-2" device="SMD-4" value=""/>
-<part name="JP1" library="SparkFun-Connectors" deviceset="USB" device="SMD" value="USBSMD"/>
+<part name="JP1" library="SparkFun-Connectors" deviceset="USB" device="PTH" value="USB-B"/>
 <part name="GND23" library="supply1" deviceset="GND" device=""/>
 <part name="P+13" library="supply1" deviceset="+12V" device=""/>
@@
 <part name="X2" library="con-molex-micro-fit-3_0" deviceset="HEADER_POS16_?" device="43045-1600"/>
 <part name="GND15" library="supply1" deviceset="GND" device=""/>
-<part name="JP2" library="SparkFun-Connectors" deviceset="M03" device="LOCK"/>
+<part name="CON_RS232" library="SparkFun-Connectors" deviceset="M03" device="LOCK"/>
 <part name="GND17" library="supply1" deviceset="GND" device=""/>
 <part name="D5" library="SparkFun-DiscreteSemi" deviceset="DIODE" device="SOD" value="BAT165"/>
 <part name="JP4" library="SparkFun-Connectors" deviceset="M05" device="JST"/>
 <part name="+3V8" library="supply1" deviceset="+3V3" device=""/>
+<part name="S3" library="SparkFun-Electromechanical" deviceset="SWITCH-MOMENTARY-2" device="SIDE_EZ" value=""/>
 </parts>
 <sheets>
@@
 <instance part="GND21" gate="1" x="436.88" y="86.36"/>
 <instance part="GND24" gate="1" x="81.28" y="43.18"/>
-<instance part="S2" gate="1" x="76.2" y="48.26" rot="R270"/>
 <instance part="P+5" gate="1" x="62.23" y="163.83"/>
 <instance part="TP3" gate="G$1" x="49.53" y="228.6" smashed="yes" rot="R180">
@@
 <instance part="X2" gate="G$1" x="415.29" y="54.61" rot="MR180"/>
 <instance part="GND15" gate="1" x="62.23" y="205.74"/>
-<instance part="JP2" gate="G$1" x="505.46" y="101.6" rot="R180"/>
+<instance part="CON_RS232" gate="G$1" x="505.46" y="101.6" rot="R180"/>
 <instance part="GND17" gate="1" x="497.84" y="95.25"/>
 <instance part="D5" gate="G$1" x="123.19" y="215.9" smashed="yes" rot="R180">
@@
 <instance part="JP4" gate="G$1" x="245.11" y="133.35" rot="MR0"/>
 <instance part="+3V8" gate="G$1" x="278.13" y="144.78"/>
+<instance part="S3" gate="G$1" x="76.2" y="48.26"/>
 </instances>
 <busses>
@@
 <pinref part="C5" gate="G$1" pin="1"/>
 <pinref part="GND14" gate="1" pin="GND"/>
-</segment>
-<segment>
-<pinref part="S2" gate="1" pin="S"/>
-<pinref part="GND24" gate="1" pin="GND"/>
 </segment>
 <segment>
@@
 </segment>
 <segment>
-<pinref part="JP2" gate="G$1" pin="3"/>
+<pinref part="CON_RS232" gate="G$1" pin="3"/>
 <pinref part="GND17" gate="1" pin="GND"/>
 <wire x1="497.84" y1="99.06" x2="497.84" y2="97.79" width="0.1524" layer="91"/>
+</segment>
+<segment>
+<pinref part="GND24" gate="1" pin="GND"/>
+<pinref part="S3" gate="G$1" pin="2"/>
+<wire x1="81.28" y1="45.72" x2="81.28" y2="48.26" width="0.1524" layer="91"/>
 </segment>
 </net>
@@
 <label x="62.23" y="48.26" size="1.778" layer="95"/>
 <wire x1="67.31" y1="48.26" x2="62.23" y2="48.26" width="0.1524" layer="91"/>
-<pinref part="S2" gate="1" pin="P"/>
+<pinref part="S3" gate="G$1" pin="1"/>
 </segment>
 <segment>
@@
 <wire x1="468.63" y1="96.52" x2="491.49" y2="96.52" width="0.1524" layer="91"/>
 <wire x1="491.49" y1="96.52" x2="491.49" y2="101.6" width="0.1524" layer="91"/>
-<pinref part="JP2" gate="G$1" pin="2"/>
+<pinref part="CON_RS232" gate="G$1" pin="2"/>
 <wire x1="491.49" y1="101.6" x2="497.84" y2="101.6" width="0.1524" layer="91"/>
 </segment>
@@
 <label x="454.66" y="101.6" size="1.778" layer="95"/>
 <pinref part="IC_232" gate="G$1" pin="T2OUT"/>
-<pinref part="JP2" gate="G$1" pin="1"/>
+<pinref part="CON_RS232" gate="G$1" pin="1"/>
 <wire x1="497.84" y1="104.14" x2="488.95" y2="104.14" width="0.1524" layer="91"/>
 <wire x1="488.95" y1="104.14" x2="488.95" y2="101.6" width="0.1524" layer="91"/>
@@
 <wire x1="340.36" y1="71.12" x2="337.82" y2="71.12" width="0.1524" layer="91"/>
 <label x="325.12" y="63.5" size="1.778" layer="95"/>
+</segment>
+<segment>
+<pinref part="Q2" gate="A" pin="I1"/>
+<wire x1="194.31" y1="184.15" x2="181.61" y2="184.15" width="0.1524" layer="91"/>
+<label x="194.31" y="184.15" size="1.778" layer="95" rot="R180"/>
 </segment>
 </net>
@@
 </segment>
 </net>
+<net name="VCC_DETECT" class="0">
+<segment>
+<pinref part="Q2" gate="A" pin="O1"/>
+<wire x1="219.71" y1="184.15" x2="232.41" y2="184.15" width="0.1524" layer="91"/>
+<label x="219.71" y="184.15" size="1.778" layer="95"/>
+</segment>
+<segment>
+<pinref part="STM32" gate="PORTB_L" pin="PB5"/>
+<wire x1="176.53" y1="125.73" x2="190.5" y2="125.73" width="0.1524" layer="91"/>
+<label x="176.53" y="125.73" size="1.778" layer="95"/>
+</segment>
+</net>

Commit message: [Board] working on rev B (routing/cleaning)
Other:
- moved on the sheet: C12
Changed lines of the file:
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@@
 <instance part="C10" gate="G$1" x="412.75" y="123.19" rot="R180"/>
 <instance part="C11" gate="G$1" x="412.75" y="113.03" rot="R180"/>
-<instance part="C12" gate="G$1" x="454.66" y="114.3" rot="MR180"/>
+<instance part="C12" gate="G$1" x="455.93" y="114.3" rot="MR180"/>
 <instance part="GND36" gate="1" x="462.28" y="109.22"/>
 <instance part="C13" gate="G$1" x="449.58" y="132.08" rot="R90"/>
@@
 <instance part="GND15" gate="1" x="62.23" y="205.74"/>
 <instance part="CON_RS232" gate="G$1" x="505.46" y="101.6" rot="R180"/>
-<instance part="GND17" gate="1" x="497.84" y="95.25"/>
+<instance part="GND17" gate="1" x="497.84" y="91.44"/>
 <instance part="D5" gate="G$1" x="123.19" y="215.9" smashed="yes" rot="R180">
 <attribute name="NAME" x="128.27" y="215.4174" size="1.778" layer="95" rot="R180"/>
@@
 <segment>
 <pinref part="C12" gate="G$1" pin="1"/>
-<wire x1="454.66" y1="109.22" x2="458.47" y2="109.22" width="0.1524" layer="91"/>
+<wire x1="455.93" y1="109.22" x2="458.47" y2="109.22" width="0.1524" layer="91"/>
 <wire x1="458.47" y1="109.22" x2="458.47" y2="111.76" width="0.1524" layer="91"/>
 <pinref part="GND36" gate="1" pin="GND"/>
@@
 <pinref part="CON_RS232" gate="G$1" pin="3"/>
 <pinref part="GND17" gate="1" pin="GND"/>
-<wire x1="497.84" y1="99.06" x2="497.84" y2="97.79" width="0.1524" layer="91"/>
+<wire x1="497.84" y1="99.06" x2="497.84" y2="93.98" width="0.1524" layer="91"/>
 </segment>
 <segment>
@@
 <pinref part="IC_232" gate="G$1" pin="V-"/>
 <pinref part="C12" gate="G$1" pin="2"/>
-</segment>
-</net>
+<wire x1="455.93" y1="116.84" x2="454.66" y2="116.84" width="0.1524" layer="91"/>
+</segment>
+</net>
